File: Digital Clock Production Hardware Rev B/Digital Clock PCB 2.0 Module Based.kicad_pcb (KiCad board)
At the start: 2 copper layers, 124.5 x 46 mm, 77 parts, among them J1 USB_C_Receptacle_USB2.0, J2 Conn_01x04, J3 Conn_01x04, Q1 C15127, Q2 C8545, SW1 SW_Push, SW2 SW_Push, U1 ESP32-S2-SOLO-2, U10 SBC18-11SURKCGKWA, U2 AMS1117-3.3, U3 74LS47, U4 74LS47, U5 SBC18-11SURKCGKWA, U6 SBC18-11SURKCGKWA, U7 74LS47, U8 74LS47, U9 SBC18-11SURKCGKWA

Commit message: Updated Hardware and folder names
Other:
- board text added: "http://NiceClock"
- board text removed: "http://NiceClock.local"
Changed lines of the file:
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@@
   (gr_line (start 269.24 126.323599) (end 146.786601 126.323599)
     (stroke (width 0.1) (type solid)) (layer "Edge.Cuts"))
-  (gr_text "http://NiceClock.local" (at 177.419 120.7262) (layer "F.SilkS")
+  (gr_text "http://NiceClock" (at 177.419 120.7262) (layer "F.SilkS")
     (effects (font (size 1 1) (thickness 0.15)))
   )
