File: Digital Clock Production Hardware Rev B/Digital Clock PCB 2.0 Module Based.kicad_sch (KiCad schematic)
At the start: 16 parts, among them J1 USB_C_Receptacle_USB2.0, J2 Conn_01x04, J3 Conn_01x04, SW1 SW_Push, SW2 SW_Push, U1 ESP32-S2-SOLO-2, U2 AMS1117-3.3

Commit message: Updated Hardware and folder names
Other:
- moved on the sheet: C1, C2, C3, R3, SW1, SW2, U1, U2
