File: Hardware/Top Plate/Nixie Clock.kicad_pcb (KiCad board)
At the start: 2 copper layers, 132.1 x 104.1 mm, 23 parts, among them J2 USB_C_Receptacle_USB2.0_16P, U6 ESP32-S2-SOLO-2

Commit message: I think these are the files I submitted to JLC
Parts:
- removed the REF** at (205.7, 62.2)
- removed the REF** at (149.9, 62.2)
- added 1v8: AMS1117-1.5, Package_TO_SOT_SMD:SOT-223-3_TabPin2, F.Cu at (229.0, 149.4)
- added 3v3: AMS1117-3.3, Package_TO_SOT_SMD:SOT-223-3_TabPin2, F.Cu at (220.5, 149.4)
- added BOOT: SW_Push, Button_Switch_SMD:SW_SPST_SKQG_WithStem, B.Cu at (148.0, 145.1)
- added C1: 10u, Capacitor_SMD:C_0603_1608Metric, F.Cu at (217.5, 144.2)
- added C13: 100n, Capacitor_SMD:C_0402_1005Metric, B.Cu at (122.9, 126.7)
- added C14: 100n, Capacitor_SMD:C_0402_1005Metric, B.Cu at (126.0, 126.4)
- added C15: 10u, Capacitor_SMD:C_0603_1608Metric, B.Cu at (122.9, 125.4)
- added C2: 10u, Capacitor_SMD:C_0603_1608Metric, F.Cu at (230.2, 144.2)
- added C3: 10u, Capacitor_SMD:C_0603_1608Metric, F.Cu at (225.9, 144.2)
- added C4: 10u, Capacitor_SMD:C_0603_1608Metric, F.Cu at (221.7, 144.2)
- added C5: 22u, Capacitor_SMD:C_1206_3216Metric, F.Cu at (196.5, 143.6)
- added C6: 22u, Capacitor_SMD:C_1206_3216Metric, F.Cu at (194.3, 156.0)
- added D9: SS34, Diode_SMD:D_SMA, F.Cu at (189.2, 154.8)
- added J1: Conn_01x04_Socket, Connector_PinHeader_2.54mm:PinHeader_1x04_P2.54mm_Vertical, F.Cu at (153.7, 116.8)
- added J10: Conn_01x04_Socket, Connector_PinHeader_2.54mm:PinHeader_1x04_P2.54mm_Vertical, F.Cu at (126.5, 149.0)
- added J3: Conn_01x04_Socket, Connector_PinHeader_2.54mm:PinHeader_1x04_P2.54mm_Vertical, F.Cu at (153.7, 157.5)
- added J4: Conn_01x04_Pin, Connector_PinHeader_2.54mm:PinHeader_1x04_P2.54mm_Vertical_SMD_Pin1Left, B.Cu at (149.9, 63.5)
- added J5: Conn_01x04_Pin, Connector_PinHeader_2.54mm:PinHeader_1x04_P2.54mm_Vertical_SMD_Pin1Left, B.Cu at (205.7, 63.5)
- added J6: Conn_01x04_Pin, Connector_PinHeader_2.54mm:PinHeader_1x04_P2.54mm_Vertical_SMD_Pin1Left, B.Cu at (149.9, 104.1)
- added J7: Conn_01x04_Pin, Connector_PinHeader_2.54mm:PinHeader_1x04_P2.54mm_Vertical_SMD_Pin1Left, B.Cu at (205.7, 104.1)
- added J8: Conn_01x04_Socket, Connector_PinHeader_2.54mm:PinHeader_1x04_P2.54mm_Vertical, F.Cu at (209.5, 157.5)
- added J9: Conn_01x04_Socket, Connector_PinHeader_2.54mm:PinHeader_1x04_P2.54mm_Vertical, F.Cu at (209.5, 116.8)
- added JP1: Jumper_2_Bridged, Resistor_SMD:R_0402_1005Metric_Pad0.72x0.64mm_HandSolder, F.Cu at (196.7, 157.5)
- added L1: 22u, Inductor_SMD:L_7.3x7.3_H3.5, F.Cu at (189.2, 146.9)
- added R3: 100k, Resistor_SMD:R_0402_1005Metric, F.Cu at (195.5, 151.6)
- added R4: 3k, Resistor_SMD:R_0402_1005Metric, F.Cu at (195.5, 149.9)
- added R7: 10k, Resistor_SMD:R_0402_1005Metric, B.Cu at (124.8, 126.4)
- added REF**: TestPoint_Pad_D1.5mm, TestPoint:TestPoint_Pad_D1.5mm, F.Cu at (223.8, 138.7)
- added RST: SW_Push, Button_Switch_SMD:SW_SPST_SKQG_WithStem, B.Cu at (131.7, 124.0)
- added U9: MT3608, Package_TO_SOT_SMD:SOT-23-6, F.Cu at (194.9, 146.9)
- U1, U2, U3, U4: footprint Indicator-Tube:IV-12 -> Indicator-Tube:IV-12 (From Real Measurements)
- U5: footprint Package_LCC:PLCC-28 -> Package_LCC:PLCC-44
- moved D8 176.4 mm to (220.2, 138.7), turned to 180 degrees
- moved D7 174.3 mm to (216.7, 138.7), turned to 180 degrees
- moved D6 155.4 mm to (194.8, 138.7), turned to 180 degrees
- moved D5 150.6 mm to (191.3, 138.7), turned to 180 degrees
- moved D4 127.0 mm to (164.3, 138.7), turned to 180 degrees
- moved D3 125.3 mm to (160.8, 138.7), turned to 180 degrees
- moved D2 108.3 mm to (138.9, 138.7), turned to 180 degrees
- moved D1 107.4 mm to (135.4, 138.7), turned to 180 degrees
- moved U5 12.8 mm to (177.3, 96.6)
Connections:
- PD1 pad 1: (no net) -> +3V3
- PD1 pad 2: (no net) -> GND
- PD1 pad 3: (no net) -> GND
- PD1 pad 4: (no net) -> SDA
- PD1 pad 5: (no net) -> +3V3
- PD1 pad 6: (no net) -> SCL
- U1 pad 1: E -> E4
- U1 pad 10: F -> F4
- U1 pad 4: Grid1 -> +GRID
- U1 pad 5: D -> D4
- U1 pad 6: C -> C4
- U1 pad 7: B -> B4
- U1 pad 8: A -> A4
- U1 pad 9: G -> G4
- U2 pad 1: E -> E3
- U2 pad 10: F -> F3
- U2 pad 4: Grid2 -> +GRID
- U2 pad 5: D -> D3
- U2 pad 6: C -> C3
- U2 pad 7: B -> B3
- U2 pad 8: A -> A3
- U2 pad 9: G -> G3
- U3 pad 1: E -> E2
- U3 pad 10: F -> F2
- U3 pad 4: Grid3 -> +GRID
- U3 pad 5: D -> D2
- U3 pad 6: C -> C2
- U3 pad 7: B -> B2
- U3 pad 8: A -> A2
- U3 pad 9: G -> G2
- U4 pad 1: E -> E1
- U4 pad 10: F -> F1
- U4 pad 4: Grid4 -> +GRID
- U4 pad 5: D -> D1
- U4 pad 6: C -> C1
- U4 pad 7: B -> B1
- U4 pad 8: A -> A1
- U4 pad 9: G -> G1
- U5 pad 10: unconnected-(U5-HV13-Pad10) -> F4
- U5 pad 11: unconnected-(U5-HV12-Pad11) -> E4
- U5 pad 12: unconnected-(U5-HV11-Pad12) -> D4
- U5 pad 13: BLANK -> C4
- U5 pad 14: GND -> B3
- U5 pad 15: CLK -> A3
- U5 pad 16: STROBE -> G3
- U5 pad 17: unconnected-(U5-HV10-Pad17) -> F3
- U5 pad 18: unconnected-(U5-HV9-Pad18) -> (no net)
- U5 pad 19: unconnected-(U5-HV8-Pad19) -> E3
- U5 pad 20: F -> D3
- U5 pad 21: G -> STROBE
- U5 pad 22: A -> GND
- U5 pad 23: B -> CLK
- U5 pad 24: C -> ~{Latch_EN}
- U5 pad 25: D -> C3
- U5 pad 26: E -> B2
- U5 pad 27: Data IN -> A2
- U5 pad 28: +3V3 -> (no net)
- U5 pad 6: unconnected-(U5-HV17-Pad6) -> (no net)
- U5 pad 7: unconnected-(U5-HV16-Pad7) -> B4
- U5 pad 8: unconnected-(U5-HV15-Pad8) -> A4
- U5 pad 9: unconnected-(U5-HV14-Pad9) -> G4
- U6 pad 11: CLK -> unconnected-(U6-IO18-Pad11)
- U6 pad 24: unconnected-(U6-IO33-Pad24) -> SCL
- U6 pad 25: unconnected-(U6-IO34-Pad25) -> SDA
- U6 pad 27: Net-(U6-IO0) -> BOOT
- U6 pad 28: unconnected-(U6-IO35-Pad28) -> Data IN
- U6 pad 29: unconnected-(U6-IO36-Pad29) -> CLK
- U6 pad 31: unconnected-(U6-IO38-Pad31) -> STROBE
- U6 pad 32: unconnected-(U6-IO39-Pad32) -> ~{Latch_EN}
- U6 pad 38: SCL -> unconnected-(U6-IO2-Pad38)
- U6 pad 39: SDA -> unconnected-(U6-IO1-Pad39)
- U6 pad 6: BLANK -> unconnected-(U6-IO6-Pad6)
- U6 pad 7: STROBE -> unconnected-(U6-IO7-Pad7)
- U6 pad 9: Data IN -> unconnected-(U6-IO16-Pad9)
Routing:
- net +3V3: track 0.00 -> 231.7 mm, vias 0 -> 6
- net +GRID: track 0.00 -> 209.4 mm, vias 0 -> 2
- net D: track 166.3 -> 0.00 mm, vias 6 -> 0
- net ~{Latch_EN}: track 0.00 -> 153.8 mm, vias 0 -> 1
- net C: track 145.0 -> 0.00 mm, vias 6 -> 0
- net +5V: track 0.00 -> 143.6 mm, vias 0 -> 1
- net +HEATER: track 0.00 -> 143.4 mm
- net E: track 139.4 -> 0.00 mm, vias 4 -> 0
- net CLK: track 10.7 -> 149.1 mm
- net STROBE: track 11.2 -> 143.8 mm
- net B: track 126.4 -> 0.00 mm, vias 6 -> 0
- net A: track 113.9 -> 0.00 mm, vias 6 -> 0
- net Data IN: track 0.00 -> 108.8 mm, vias 0 -> 2
- net G: track 108.3 -> 0.00 mm, vias 6 -> 0
- net F: track 105.7 -> 0.00 mm, vias 4 -> 0
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Other:
- outline, holes or cut-outs redrawn
- board text added: "Ambient Light BH1730"
- board text added: "Clocks Signals"
- board text added: "Data Power"
- board text added: "GND RX TX +3v3"
- board text added: "JLCJLCJLCJLC"
- board text added: "Mechanical"
