File: Hardware/Top Plate/Nixie Clock.kicad_sch (KiCad schematic)
At the start: 8 parts, among them J1 Conn_01x18_Pin, J3 Conn_01x18_Pin

Commit message: I think these are the files I submitted to JLC
Parts:
- removed J1, J3: Conn_01x18_Pin, Connector_PinHeader_2.54mm:PinHeader_1x18_P2.54mm_Vertical_SMD_Pin1Left, symbol Connector:Conn_01x18_Pin
- removed U5: ~, Package_LCC:PLCC-28, symbol Indicator_Tube:HV5812
- added J4, J5, J6, J7: Conn_01x04_Pin, Connector_PinHeader_2.54mm:PinHeader_1x04_P2.54mm_Vertical_SMD_Pin1Left, symbol Connector:Conn_01x04_Pin
- added U5: ~, Package_LCC:PLCC-44, symbol Indicator_Tube:HV518
- U1, U2, U3, U4: footprint Indicator-Tube:IV-12 -> Indicator-Tube:IV-12 (From Real Measurements)
Connections:
- net Grid1 is gone; now on net +GRID: U1.4 (Grid)
- net Grid2 is gone; now on net +GRID: U2.4 (Grid)
- net Grid3 is gone; now on net +GRID: U3.4 (Grid)
- net Grid4 is gone; now on net +GRID: U4.4 (Grid)
- net +3V3: now also PD1.1 (VCC), PD1.5 (DVI), J4.3 (Pin_3), J7.2 (Pin_2), U5.44 (Vdd); no longer PD1. (VCC)
- net +GRID: now also J7.3 (Pin_3), U5.1 (Vpp)
- net +HEATER: now also J7.4 (Pin_4)
- net A1: now also U4.8 (a), U5.36 (HVOUT7)
- net A2: now also U3.8 (a), U5.27 (HVOUT14)
- net A3: now also U2.8 (a), U5.15 (HVOUT21)
- net A4: now also U1.8 (a), U5.8 (HVOUT28)
- net B1: now also U4.7 (b), U5.35 (HVOUT8)
- net B2: now also U3.7 (b), U5.26 (HVOUT15)
- net B3: now also U2.7 (b), U5.14 (HVOUT22)
- net B4: now also U1.7 (b), U5.7 (HVOUT29)
- net C1: now also U4.6 (c), U5.41 (HVOUT2)
- net C2: now also U3.6 (c), U5.34 (HVOUT9)
- net C3: now also U2.6 (c), U5.25 (HVOUT16)
- net C4: now also U1.6 (c), U5.13 (HVOUT23)
- net CLK: now also J5.3 (Pin_3), U5.23 (CLK)
- net D1: now also U4.5 (d), U5.40 (HVOUT3)
- net D2: now also U3.5 (d), U5.33 (HVOUT10)
- net D3: now also U2.5 (d), U5.20 (HVOUT17)
- net D4: now also U1.5 (d), U5.12 (HVOUT24)
- net Data IN: now also J7.1 (Pin_1), U5.43 (Data_In)
- net E1: now also U4.1 (e), U5.39 (HVOUT4)
- net E2: now also U3.1 (e), U5.32 (HVOUT11)
- net E3: now also U2.1 (e), U5.19 (HVOUT18)
- net E4: now also U1.1 (e), U5.11 (HVOUT25)
- net F1: now also U4.10 (f), U5.38 (HVOUT5)
- net F2: now also U3.10 (f), U5.31 (HVOUT12)
- net F3: now also U2.10 (f), U5.17 (HVOUT19)
- net F4: now also U1.10 (f), U5.10 (HVOUT26)
- net G1: now also U4.9 (g), U5.37 (HVOUT6)
- net G2: now also U3.9 (g), U5.30 (HVOUT13)
- net G3: now also U2.9 (g), U5.16 (HVOUT20)
- net G4: now also U1.9 (g), U5.9 (HVOUT27)
- net GND: now also PD1.2 (INT), PD1.3 (GND), J4.4 (Pin_4), J5.2 (Pin_2), J6.1 (Pin_1), J6.2 (Pin_2), J6.3 (Pin_3), J6.4 (Pin_4), U5.22 (GND); no longer PD1. (VCC)
- net SCL: now also PD1.6 (SCL), J4.1 (Pin_1); no longer PD1. (VCC)
- net SDA: now also PD1.4 (SDA), J4.2 (Pin_2); no longer PD1. (VCC)
- net STROBE: now also J5.1 (Pin_1), U5.21 (Strobe)
- removed net A: U1.8 (a), U2.8 (a), U3.8 (a), U4.8 (a)
- removed net B: U1.7 (b), U2.7 (b), U3.7 (b), U4.7 (b)
- removed net C: U1.6 (c), U2.6 (c), U3.6 (c), U4.6 (c)
- removed net D: U1.5 (d), U2.5 (d), U3.5 (d), U4.5 (d)
- removed net E: U1.1 (e), U2.1 (e), U3.1 (e), U4.1 (e)
- removed net F: U1.10 (f), U2.10 (f), U3.10 (f), U4.10 (f)
- removed net G: U1.9 (g), U2.9 (g), U3.9 (g), U4.9 (g)
- new net ~{Latch_EN}: J5.4 (Pin_4), U5.24 (~{Latch_EN})
- no-connect marks 1 -> 5
