File: Hardware/Top Plate/untitled.kicad_sch (KiCad schematic)
At the start: 13 parts, among them J2 USB_C_Receptacle_USB2.0_16P, SW1 SW_Push, U6 ESP32-S2-SOLO-2

Commit message: I think these are the files I submitted to JLC
Parts:
- removed SW1: SW_Push, symbol Switch:SW_Push
- added C1, C15, C2, C3, C4: 10u, Capacitor_SMD:C_0603_1608Metric, symbol Device:C
- added C13: 100n, Capacitor_SMD:C_0402_1005Metric, symbol Device:C
- added C14: 100n, Capacitor_SMD:C_0402_1005Metric, symbol Device:C_Small
- added J1, J10, J3, J8, J9: Conn_01x04_Socket, Connector_PinHeader_2.54mm:PinHeader_1x04_P2.54mm_Vertical, symbol Connector:Conn_01x04_Socket
- added R7: 10k, Resistor_SMD:R_0402_1005Metric, symbol Device:R_Small
- added RST1, SW2: SW_Push, Button_Switch_SMD:SW_SPST_SKQG_WithStem, symbol Switch:SW_Push
- added U7: AMS1117-1.5, Package_TO_SOT_SMD:SOT-223-3_TabPin2, symbol Regulator_Linear:AMS1117-1.5
- added U8: AMS1117-3.3, Package_TO_SOT_SMD:SOT-223-3_TabPin2, symbol Regulator_Linear:AMS1117-3.3
Connections:
- net +3V3: now also C13.1, C15.1, C4.1, J1.2 (Pin_2), J10.4 (Pin_4), J8.3 (Pin_3), R7.2, U8.2 (VO)
- net +5V: now also C1.1, C3.1, U7.3 (VI), U8.3 (VI)
- net CLK: now also U6.29 (IO36), J9.2 (Pin_2); no longer U6.11 (IO18)
- net Data IN: now also U6.28 (IO35), J8.4 (Pin_4); no longer U6.9 (IO16)
- net GND: now also C1.2, C13.2, C14.2, C15.2, C2.2, C3.2, C4.2, J1.1 (Pin_1), J10.1 (Pin_1), J3.1 (Pin_1), J3.2 (Pin_2), J3.3 (Pin_3), J3.4 (Pin_4), J9.3 (Pin_3), RST1.2, SW2.2, U7.1 (GND), U8.1 (GND)
- net RST: now also C14.1, R7.1, RST1.1
- net RX: now also J10.2 (Pin_2)
- net SCL: now also U6.24 (IO33), J1.4 (Pin_4); no longer U6.38 (IO2)
- net SDA: now also U6.25 (IO34), J1.3 (Pin_3); no longer U6.39 (IO1)
- net STROBE: now also U6.31 (IO38), J9.4 (Pin_4); no longer U6.7 (IO7)
- net TX: now also J10.3 (Pin_3)
- net BOOT: now reaches U6.27 (IO0)
- net BOOT: now also SW2.1
- net ~{Latch_EN}: now reaches U6.32 (IO39)
- net ~{Latch_EN}: now also J9.1 (Pin_1)
- net BLANK: no longer names the net of U6.6 (IO6)
- new net +GRID: J8.2 (Pin_2)
- new net +HEATER: C2.1, J8.1 (Pin_1), U7.2 (VO)
- no-connect marks 9 -> 12
Other:
- added sheet Boost (boost.kicad_sch)
- note added: "Boot"
- note added: "Filter"
- note added: "Reset"
- note added: "Strapping"
- moved on the sheet: D1, D2, D3, D4, D5, D6, D7, D8, J2, U6
